Commit message: Added IMU and UWB nodes

File: urdf/gazebo_specific.urdf.xacro (robot description, xacro)
@@ -72,4 +72,52 @@
       </sensor>
     </gazebo>
+    <!-- IMU Sensor -->
+    <gazebo reference="imu_link">
+      <sensor type="imu" name="imu_sensor">
+        <always_on>true</always_on>
+        <update_rate>50</update_rate>
+        <imu>
+          <topic>${topic_prefix}/imu</topic>
+          <orientation>true</orientation>
+          <angular_velocity>true</angular_velocity>
+          <linear_acceleration>true</linear_acceleration>
+        </imu>
+        <plugin name="gazebo_ros_imu" filename="libgazebo_ros_imu_sensor.so
+">
+          <ros>
+            <namespace>${topic_prefix}</namespace>
+            <remapping>imu:=/imu</remapping>
+          </ros>
+          <update_rate>50.0</update_rate>
+          <body_name>imu_link</body_name>
+          <gaussian_noise>0</gaussian_noise>
+          <xyz_offset>0 0 0</xyz_offset>
+          <rpy_offset>0 0 0</rpy_offset>
+        </plugin>
+      </sensor>
+    </gazebo>
+    <!-- UWB Sensor -->
+    <gazebo reference="uwb_link">
+      <sensor type="range" name="uwb_sensor">
+        <always_on>true</always_on>
+        <update_rate>10</update_rate>
+        <visualize>true</visualize>
+        <pose>0 0 0 0 0 0</pose>
+        <range>
+          <min>0.02</min>
+          <max>10.0</max>
+          <resolution>0.01</resolution>
+        </range>
+        <plugin name="gazebo_ros_range" filename="libgazebo_ros_range.so">
+          <ros>
+            <namespace>${topic_prefix}</namespace>
+            <remapping>uwb:=/uwb</remapping>
+          </ros>
+          <update_rate>10.0</update_rate>
+          <radiation>ultrasonic</radiation>
+          <frame_name>${frame_prefix}uwb</frame_name>
+        </plugin>
+      </sensor>
+    </gazebo>
 	</xacro:macro>
 </robot>

File: urdf/turtlebot3_waffle.urdf.xacro (robot description, xacro)
@@ -167,14 +167,52 @@
     </inertial>
   </link>
+  <link name="imu_link">
+    <inertial>
+      <mass value="0.01"/>
+      <origin xyz="0 0 0" rpy="0 0 0"/>
+      <inertia ixx="0.0001" ixy="0.0" ixz="0.0" iyy="0.0001" iyz="0.0" izz="0.0001"/>
+    </inertial>
+    <visual>
+      <geometry>
+        <box size="0.030 0.009 0.020"/>
+      </geometry>
+    </visual>
+    <collision>
+      <geometry>
+        <box size="0.030 0.009 0.020"/>
+      </geometry>
+    </collision>
+  </link>
   <joint name="imu_joint" type="fixed">
     <parent link="base_link"/>
     <child link="imu_link"/>
-    <origin xyz="0.0 0 0.068" rpy="0 0 0"/>
-  </joint>
-  <link name="imu_link"/>
+    <origin xyz="0 0 0" rpy="0 0 0"/>
+  </joint>
   <joint name="scan_joint" type="fixed">
     <parent link="base_link"/>
     <child link="base_scan"/>
     <origin xyz="-0.064 0 0.122" rpy="0 0 0"/>
+  </joint>
+  <link name="uwb_link">
+    <inertial>
+      <mass value="0.01"/>
+      <origin xyz="0 0 0" rpy="0 0 0"/>
+      <inertia ixx="0.0001" ixy="0.0" ixz="0.0" iyy="0.0001" iyz="0.0" izz="0.0001"/>
+    </inertial>
+    <visual>
+      <geometry>
+        <box size="0.030 0.009 0.020"/>
+      </geometry>
+    </visual>
+    <collision>
+      <geometry>
+        <box size="0.030 0.009 0.020"/>
+      </geometry>
+    </collision>
+  </link>
+  <joint name="uwb_joint" type="fixed">
+    <parent link="base_link"/>
+    <child link="uwb_link"/>
+    <origin xyz="0.1 0 0.1" rpy="0 0 0"/>
   </joint>
   <link name="base_scan">
